File: pifire-relay-module-SSR.kicad_sch (KiCad schematic)
At the start: 25 parts, among them J1 AC Terminal, J6 RELAY/FAN Header, K1 Power Relay, K2 Auger Relay, K3 Igniter Relay, K4 Fan Relay, Q1 BC547, Q2 BC547, Q3 BC547, Q4 BC547

Commit message: Updated to V1.0.2
This version is a minor update to change 4.7k Ohm resistor values to 470 Ohms.  Some users had pointed out that the 4.7k Ohm resistors may be too large and may not allow the transistors to properly turn on.  This should fix that issue.
Parts:
- R1, R3, R5, R7: value 4.7k -> 470
Changed lines of the file:
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@@
 (kicad_sch
-	(version 20231120)
+	(version 20250114)
 	(generator "eeschema")
-	(generator_version "8.0")
+	(generator_version "9.0")
 	(paper "A4")
 	(title_block
 		(title "PiFire Relay Module")
-		(date "2024-05-10")
-		(rev "v1.0.1")
+		(date "2025-12-24")
+		(rev "v1.0.2")
 		(company "PiFire")
 		(comment 1 "https://github.com/nebhead/pifire")
 		(comment 2 "Ben Parmeter")
 	)
+	(rectangle
+		(start 17.78 90.17)
+		(end 101.6 163.83)
+		(stroke
+			(width 0)
+			(type default)
+		)
+		(fill
+			(type none)
+		)
+	)
+	(rectangle
+		(start 124.46 142.24)
+		(end 166.37 167.64)
+		(stroke
+			(width 0)
+			(type default)
+		)
+		(fill
+			(type none)
+		)
+	)
+	(rectangle
+		(start 102.87 15.24)
+		(end 186.69 88.9)
+		(stroke
+			(width 0)
+			(type default)
+		)
+		(fill
+			(type none)
+		)
+	)
+	(rectangle
+		(start 17.78 15.24)
+		(end 101.6 88.9)
+		(stroke
+			(width 0)
+			(type default)
+		)
+		(fill
+			(type none)
+		)
+	)
+	(rectangle
+		(start 180.34 106.68)
+		(end 222.25 137.16)
+		(stroke
+			(width 0)
+			(type default)
+		)
+		(fill
+			(type none)
+		)
+	)
+	(rectangle
+		(start 124.46 106.68)
+		(end 166.37 137.16)
+		(stroke
+			(width 0)
+			(type default)
+		)
+		(fill
+			(type none)
+		)
+	)
+	(rectangle
+		(start 187.96 15.24)
+		(end 271.78 88.9)
+		(stroke
+			(width 0)
+			(type default)
+		)
+		(fill
+			(type none)
+		)
+	)
+	(text "Fan Relay"
+		(exclude_from_sim no)
+		(at 196.596 18.288 0)
+		(effects
+			(font
+				(size 1.27 1.27)
+			)
+		)
+	)
+	(text "Power Relay"
+		(exclude_from_sim no)
+		(at 25.654 93.726 0)
+		(effects
+			(font
+				(size 1.27 1.27)
+			)
+		)
+	)
+	(text "Fuses (F1-3): \n  Littelfuse 2A Slow Blow (39212000000)\n  https://www.digikey.com/en/products/detail/littelfuse-inc/39212000000/653505"
+		(exclude_from_sim no)
+		(at 17.78 176.784 0)
+		(effects
+			(font
+				(size 1.27 1.27)
+				(thickness 0.254)
+				(bold yes)
+			)
+			(justify left)
+		)
+	)
+	(text "AC Terminal Block"
+		(exclude_from_sim no)
+		(at 137.668 144.78 0)
+		(effects
+			(font
+				(size 1.27 1.27)
+			)
+		)
+	)
+	(text "Auger Relay"
+		(exclude_from_sim no)
+		(at 25.146 18.034 0)
+		(effects
+			(font
+				(size 1.27 1.27)
+			)
+		)
+	)
+	(text "Relay/Fan Board Header"
+		(exclude_from_sim no)
+		(at 153.67 108.712 0)
+		(effects
+			(font
+				(size 1.27 1.27)
+			)
+		)
+	)
+	(text "Relays (K1-4): \n  G3MB-202P  5V 2A SSR  \n  https://www.amazon.com/dp/B082F8C1LX"
+		(exclude_from_sim no)
+		(at 17.526 169.672 0)
+		(effects
+			(font
+				(size 1.27 1.27)
+				(thickness 0.254)
+				(bold yes)
+			)
+			(justify left)
+			(href "https://www.amazon.com/dp/B082F8C1LX")
+		)
+	)
+	(text "Mounting Holes"
+		(exclude_from_sim no)
+		(at 188.722 108.966 0)
+		(effects
+			(font
+				(size 1.27 1.27)
+			)
+		)
+	)
+	(text "Igniter Relay"
+		(exclude_from_sim no)
+		(at 110.49 18.288 0)
+		(effects
+			(font
+				(size 1.27 1.27)
+			)
+		)
+	)
 	(junction
 		(at 41.91 120.65)
@@
 		)
 	)
-	(rectangle
-		(start 17.78 90.17)
-		(end 101.6 163.83)
-		(stroke
-			(width 0)
-			(type default)
-		)
-		(fill
-			(type none)
-		)
-	)
-	(rectangle
-		(start 124.46 142.24)
-		(end 166.37 167.64)
-		(stroke
-			(width 0)
-			(type default)
-		)
-		(fill
-			(type none)
-		)
-	)
-	(rectangle
-		(start 102.87 15.24)
-		(end 186.69 88.9)
-		(stroke
-			(width 0)
-			(type default)
-		)
-		(fill
-			(type none)
-		)
-	)
-	(rectangle
-		(start 17.78 15.24)
-		(end 101.6 88.9)
-		(stroke
-			(width 0)
-			(type default)
-		)
-		(fill
-			(type none)
-		)
-	)
-	(rectangle
-		(start 180.34 106.68)
-		(end 222.25 137.16)
-		(stroke
-			(width 0)
-			(type default)
-		)
-		(fill
-			(type none)
-		)
-	)
-	(rectangle
-		(start 124.46 106.68)
-		(end 166.37 137.16)
-		(stroke
-			(width 0)
-			(type default)
-		)
-		(fill
-			(type none)
-		)
-	)
-	(rectangle
-		(start 187.96 15.24)
-		(end 271.78 88.9)
-		(stroke
-			(width 0)
-			(type default)
-		)
-		(fill
-			(type none)
-		)
-	)
 	(image
 		(at 276.86 173.99)
@@
 		)
 	)
-	(text "Fan Relay"
-		(exclude_from_sim no)
-		(at 196.596 18.288 0)
-		(effects
-			(font
-				(size 1.27 1.27)
-			)
-		)
-	)
-	(text "Power Relay"
-		(exclude_from_sim no)
-		(at 25.654 93.726 0)
-		(effects
-			(font
-				(size 1.27 1.27)
-			)
-		)
-	)
-	(text "Fuses (F1-3): \n  Littelfuse 2A Slow Blow (39212000000)\n  https://www.digikey.com/en/products/detail/littelfuse-inc/39212000000/653505"
-		(exclude_from_sim no)
-		(at 17.78 176.784 0)
-		(effects
-			(font
-				(size 1.27 1.27)
-				(thickness 0.254)
-				(bold yes)
-			)
-			(justify left)
-		)
-	)
-	(text "AC Terminal Block"
-		(exclude_from_sim no)
-		(at 137.668 144.78 0)
-		(effects
-			(font
-				(size 1.27 1.27)
-			)
-		)
-	)
-	(text "Auger Relay"
-		(exclude_from_sim no)
-		(at 25.146 18.034 0)
-		(effects
-			(font
-				(size 1.27 1.27)
-			)
-		)
-	)
-	(text "Relay/Fan Board Header"
-		(exclude_from_sim no)
-		(at 153.67 108.712 0)
-		(effects
-			(font
-				(size 1.27 1.27)
-			)
-		)
-	)
-	(text "Relays (K1-4): \n  G3MB-202P  5V 2A SSR  \n  https://www.amazon.com/dp/B082F8C1LX"
-		(exclude_from_sim no)
-		(at 17.526 169.672 0)
-		(effects
-			(font
-				(size 1.27 1.27)
-				(thickness 0.254)
-				(bold yes)
-			)
-			(justify left)
-			(href "https://www.amazon.com/dp/B082F8C1LX")
-		)
-	)
-	(text "Mounting Holes"
-		(exclude_from_sim no)
-		(at 188.722 108.966 0)
-		(effects
-			(font
-				(size 1.27 1.27)
-			)
-		)
-	)
-	(text "Igniter Relay"
-		(exclude_from_sim no)
-		(at 110.49 18.288 0)
-		(effects
-			(font
-				(size 1.27 1.27)
-			)
-		)
-	)
 	(global_label "AUG"
 		(shape input)
@@
 		(on_board yes)
 		(dnp no)
-		(fields_autoplaced yes)
 		(property "Reference" "R5"
 			(at 204.47 43.18 90)
@@
 			)
 		)
-		(property "Value" "4.7k"
-			(at 204.47 45.72 90)
+		(property "Value" "470"
+			(at 204.724 45.974 90)
 			(effects
 				(font
@@
 			)
 		)
-		(property "Value" "4.7k"
+		(property "Value" "470"
 			(at 34.29 116.84 90)
 			(effects
@@
 			)
 		)
-		(property "Value" "4.7k"
+		(property "Value" "470"
 			(at 119.38 46.99 90)
 			(effects
@@
 			)
 		)
-		(property "Value" "4.7k"
+		(property "Value" "470"
 			(at 35.56 46.99 90)
 			(effects
@@
 		)
 	)
+	(embedded_fonts no)
 )
