File: pifire-relay-module-SSR.kicad_pcb (KiCad board)
At the start: 2 copper layers, 65 x 46 mm, 25 parts, among them J1 AC Terminal, J6 RELAY/FAN Header, K1 Power Relay, K2 Auger Relay, K3 Igniter Relay, K4 Fan Relay, Q1 BC547, Q2 BC547, Q3 BC547, Q4 BC547

Commit message: Updated to V1.0.2
This version is a minor update to change 4.7k Ohm resistor values to 470 Ohms.  Some users had pointed out that the 4.7k Ohm resistors may be too large and may not allow the transistors to properly turn on.  This should fix that issue.
Parts:
- R1, R3, R5, R7: value 4.7k -> 470
Other:
- board text added: "PiFire Relay Module SSR v1.0.2"
- board text removed: "(L)"
- board text removed: "(N)"
- board text removed: "PiFire Relay Module SSR v1.0.1"

Commit message: Updated v1.0.2 December on backside
Other:
- board text added: "v1.0.2 | December 2025 | Ben Parmeter"
- board text removed: "v1.0.1 | May 2024 | Ben Parmeter"
Changed lines of the file:
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@@
 		)
 	)
-	(gr_text "v1.0.1 | May 2024 | Ben Parmeter"
+	(gr_text "v1.0.2 | December 2025 | Ben Parmeter"
 		(at 65 36.5 90)
 		(layer "B.SilkS")
@@
 			(justify left bottom mirror)
 		)
-		(render_cache "v1.0.1 | May 2024 | Ben Parmeter" 90
+		(render_cache "v1.0.2 | December 2025 | Ben Parmeter" 90
 			(polygon
 				(pts
